File: CCLoad.kicad_pcb (KiCad board)
At the start: 2 copper layers, 100 x 50 mm, 5 parts, among them U1 STUSB4500

Commit message: finished board, generated output files
Parts:
- removed U1: STUSB4500, CCLoad:QFN-24_EP_4x4_Pitch0.5mm
- added BT101: Battery_Cell, Battery:BatteryHolder_Keystone_1060_1x2032, B.Cu at (116.9, 102.5)
- added C101: 1uF, Capacitor_SMD:C_0805_2012Metric_Pad1.15x1.40mm_HandSolder, B.Cu at (172.1, 120.0)
- added C102: 10uF, Capacitor_Tantalum_SMD:CP_EIA-3216-12_Kemet-S_Pad1.58x1.35mm_HandSolder, B.Cu at (161.9, 120.0)
- added C103: 10uF, Capacitor_Tantalum_SMD:CP_EIA-3216-12_Kemet-S_Pad1.58x1.35mm_HandSolder, B.Cu at (144.1, 120.0)
- added C104: 1uF, Capacitor_SMD:C_0805_2012Metric_Pad1.15x1.40mm_HandSolder, B.Cu at (170.6, 95.1)
- added C105: 100nF, Capacitor_SMD:C_0805_2012Metric_Pad1.15x1.40mm_HandSolder, B.Cu at (168.3, 108.2)
- added D101: LED, LED_SMD:LED_0805_2012Metric_Pad1.15x1.40mm_HandSolder, F.Cu at (145.9, 122.6)
- added J101: BANANA, CCLoad:Binding_Post_Caltest_CT2234, F.Cu at (182.8, 88.9)
- added J102: BANANA, CCLoad:Binding_Post_Caltest_CT2234, F.Cu at (182.9, 116.2)
- added J103: MOLEX, Connector_PinHeader_2.54mm:PinHeader_1x02_P2.54mm_Vertical, F.Cu at (196.8, 101.2)
- added J104: BTS117, CCLoad:BTS117_outboard, B.Cu at (182.6, 101.6)
- added J105: SCREW_TERMINAL, Connector_Molex:Molex_KK-254_AE-6410-02A_1x02_P2.54mm_Vertical, F.Cu at (154.3, 81.0)
- added J106: MOLEX, Connector_PinHeader_2.54mm:PinHeader_1x02_P2.54mm_Vertical, F.Cu at (165.1, 81.0)
- added JP101: Jumper_2_Bridged, Jumper:SolderJumper-2_P1.3mm_Bridged_RoundedPad1.0x1.5mm, B.Cu at (132.1, 116.8)
- added JP102: Jumper_3_Open, Jumper:SolderJumper-3_P1.3mm_Bridged12_RoundedPad1.0x1.5mm, B.Cu at (146.1, 99.1)
- added JP103: Jumper_3_Open, Jumper:SolderJumper-3_P1.3mm_Bridged12_RoundedPad1.0x1.5mm, B.Cu at (146.1, 104.2)
- added JP104: Jumper_2_Open, Jumper:SolderJumper-2_P1.3mm_Open_RoundedPad1.0x1.5mm, B.Cu at (135.9, 116.8)
- added R101: 162k, Resistor_SMD:R_0805_2012Metric_Pad1.15x1.40mm_HandSolder, B.Cu at (132.1, 122.3)
- added R102: 330R, Resistor_SMD:R_0805_2012Metric_Pad1.15x1.40mm_HandSolder, B.Cu at (139.7, 122.3)
- added R103: 82k, Resistor_SMD:R_0805_2012Metric_Pad1.15x1.40mm_HandSolder, B.Cu at (135.9, 122.3)
- added R104: 100R, Resistor_SMD:R_0805_2012Metric_Pad1.15x1.40mm_HandSolder, B.Cu at (170.6, 108.2)
- added R105: 0R, Resistor_SMD:R_0805_2012Metric_Pad1.15x1.40mm_HandSolder, B.Cu at (165.9, 108.2)
- added R106: 0.1R, Resistor_SMD:R_2512_6332Metric_Pad1.52x3.35mm_HandSolder, B.Cu at (188.7, 108.3)
- added R107: 100R, Resistor_SMD:R_0805_2012Metric_Pad1.15x1.40mm_HandSolder, B.Cu at (150.5, 116.7)
- added R108: 0.1R, Resistor_SMD:R_2512_6332Metric_Pad1.52x3.35mm_HandSolder, B.Cu at (192.8, 108.3)
- added R109: 10k, Resistor_SMD:R_0805_2012Metric_Pad1.15x1.40mm_HandSolder, B.Cu at (165.9, 95.1)
- added R110: 10k, Resistor_SMD:R_0805_2012Metric_Pad1.15x1.40mm_HandSolder, B.Cu at (168.3, 95.1)
- added RV101: 10k, Potentiometer_THT:Potentiometer_Alps_RK09K_Single_Vertical, F.Cu at (142.2, 99.9)
- added RV102: 1k, Potentiometer_SMD:Potentiometer_Bourns_3314J_Vertical, B.Cu at (168.1, 90.0)
- added SW101: SW_DP3T, CCLoad:SW_DP3T_ALPS_SSSS223600, F.Cu at (152.5, 122.5)
- added U101: HT7533-1 (3V3), Package_TO_SOT_SMD:SOT-89-3_Handsoldering, B.Cu at (167.0, 119.9)
- added U102: CJ431, Package_TO_SOT_SMD:SOT-23, B.Cu at (140.3, 116.8)
- added U103: MCP6002-xP, Package_SO:SOIC-8_3.9x4.9mm_P1.27mm, B.Cu at (168.3, 101.6)
- H101: renamed from H1; footprint MountingHole:MountingHole_3.7mm_Pad_Via -> MountingHole:MountingHole_3.7mm_Pad
- H102: renamed from H2; footprint MountingHole:MountingHole_3.7mm_Pad_Via -> MountingHole:MountingHole_3.7mm_Pad
- H103: renamed from H3; footprint MountingHole:MountingHole_3.7mm_Pad_Via -> MountingHole:MountingHole_3.7mm_Pad
- H104: renamed from H4; footprint MountingHole:MountingHole_3.7mm_Pad_Via -> MountingHole:MountingHole_3.7mm_Pad
- moved H103 127.8 mm to (196.8, 82.3)
- moved H104 127.8 mm to (196.8, 122.8)
- moved H101 127.8 mm to (106.3, 82.3)
- moved H102 127.8 mm to (106.3, 122.8)
Routing:
- net VDD: track 0.00 -> 63.7 mm
- net Net-(C103-Pad1): track 0.00 -> 60.7 mm
- net /BATTERY+: track 0.00 -> 51.3 mm
- net Net-(JP101-Pad1): track 0.00 -> 44.0 mm
- net Net-(J104-Pad1): track 0.00 -> 36.7 mm, vias 0 -> 2
- net /MEASURE: track 0.00 -> 31.5 mm
- net Net-(RV101-Pad2): track 0.00 -> 27.9 mm
- net Net-(J104-Pad2): track 0.00 -> 26.1 mm, vias 0 -> 2
- net Net-(RV102-Pad2): track 0.00 -> 14.2 mm
- net +2V5: track 0.00 -> 14.0 mm
- net /SENSE: track 0.00 -> 11.8 mm
- net Net-(D101-Pad2): track 0.00 -> 9.46 mm
- net Net-(C102-Pad1): track 0.00 -> 9.39 mm
- net Net-(D101-Pad1): track 0.00 -> 7.10 mm, vias 0 -> 1
- net Net-(R110-Pad2): track 0.00 -> 6.82 mm
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- added copper zone on B.Cu, net GND
- added copper zone on F.Cu, net GND
Other:
- outline, holes or cut-outs redrawn
- board text added: "+"
- board text added: "30V MAX PLEASE"
- board text added: "BATTERY"
- board text added: "CASE CAN GET"
- board text added: "GND"
- board text added: "LOAD"
- board text added: "M. KALINOWSKI CC LOAD REV. A NOV 2019"
- board text added: "MEASURE"
- board text added: "MEASURE OUT 0.1V per 1A of input current"
- board text added: "OFF"
- board text added: "Select BATTERY power for load voltage smaller than 3V"
